File: Board/PAMI.kicad_sch (KiCad schematic)
At the start: 48 parts, among them J1 Conn_01x04_Pin, SW1 Conn_01x03_Pin, U1 BD9P135MUF-CE2, U2 STM32L031F6Px, U3 TC78H621FNG

Commit message: Update WE before coupe
Parts:
- RQSL1: value 1k -> 10k
Changed lines of the file:
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@@
       (effects (font (size 1.27 1.27)))
     )
-    (property "Value" "1k" (at 191.77 137.16 90)
+    (property "Value" "10k" (at 191.77 137.16 90)
       (effects (font (size 1.27 1.27)))
     )
